File: Universal Charger.kicad_pcb (KiCad board)
At the start: 2 copper layers, 25 x 39 mm, 38 parts, among them J1 Conn_01x02_Pin, J2 Conn_01x02_Pin, J3 USB_C_Receptacle_USB2.0_16P, J4 Conn_BAT, J5 Conn_01x02_Pin, J6 Conn_01x02_Pin, J7 Conn_01x02_Pin, U6 TP4056, U8 TPS63001, U9 TPS63002

Commit message: Implemented the Universak charger fully including Gerber
Routing:
- net +5V: track 27.2 -> 33.6 mm, vias 2 -> 3
- net GND: track 10.5 -> 13.4 mm, vias 28 -> 32
- net Net-(U8-EN): track 3.65 -> 5.50 mm
- net Net-(U9-EN): track 3.58 -> 5.11 mm
Other:
- board text added: "3V3"
- board text added: "5V"
- board text added: "CHRG"
- board text added: "DONE"
- board text added: "GND"
- board text added: "NTC"
- board text added: "VBAT"
